File: southpaw/vanapad.kicad_pcb (KiCad board)
At the start: 2 copper layers, 328.6 x 81 mm, 145 parts, among them J1 Battery JST, J2 External Power Switch, J3 Battery THT, SW1 MX_SW_HS, SW10 MX_SW_HS, SW11 MX_SW_HS, SW12 MX_SW_HS, SW13 MX_SW_HS, SW14 MX_SW_HS, SW15 MX_SW_HS, SW16 MX_SW_HS, SW17 MX_SW_HS, SW18 MX_SW_HS, SW19 MX_SW_HS, SW2 MX_SW_HS, SW20 MX_SW_HS, SW21 MX_SW_HS, SW22 MX_SW_HS, SW23 MX_SW_HS, SW24 MX_SW_HS, SW25 MX_SW_HS, SW26 MX_SW_HS, SW27 MX_SW_HS, SW28 MX_SW_HS, SW29 MX_SW_HS, SW3 MX_SW_HS, SW30 MX_SW_HS, SW31 MX_SW_HS, SW32 MX_SW_HS, SW33 MX_SW_HS, SW34 MX_SW_HS, SW35 MX_SW_HS, SW36 MX_SW_HS, SW37 MX_SW_HS, SW38 MX_SW_HS, SW39 MX_SW_HS, SW4 MX_SW_HS, SW40 MX_SW_HS, SW41 MX_SW_HS, SW42 MX_SW_HS, SW43 MX_SW_HS, SW44 MX_SW_HS, SW45 MX_SW_HS, SW46 MX_SW_HS, SW47 MX_SW_HS, SW48 MX_SW_HS, SW49 MX_SW_HS, SW5 MX_SW_HS, SW50 MX_SW_HS, SW51 MX_SW_HS, SW52 MX_SW_HS, SW53 MX_SW_HS, SW54 MX_SW_HS, SW55 MX_SW_HS, SW56 MX_SW_HS, SW57 MX_SW_HS, SW58 MX_SW_HS, SW59 MX_SW_HS, SW6 MX_SW_HS, SW60 MX_SW_HS, SW61 MX_SW_HS, SW62 On-Board Power Switch, SW63 SW_Push, SW64 MX_SW_HS, SW65 MX_SW_HS, SW66 MX_SW_HS, SW67 MX_SW_HS, SW7 MX_SW_HS, SW8 MX_SW_HS, SW9 MX_SW_HS, U1 nice_nano

Commit message: fix alternative bottom row routing
Parts:
- SW60, SW61: footprint PCM_marbastlib-mx:SW_MX_HS_1u -> PCM_marbastlib-mx:SW_MX_HS_CPG151101S11_1.5u
Connections:
- SW60 pad 1: c1 -> c3
- SW61 pad 1: c3 -> c1
Routing:
- net c3: track 261.4 -> 266.8 mm

Commit message: make vanapad pcb compatible with mirrored case
Parts:
- moved H5 14.3 mm to (354.2, 92.9)
Changed lines of the file:
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@@
 		(fp_arc
 			(start 15.28125 7.500001)
-			(mid 15.134806 7.853571)
+			(mid 15.1348 7.853536)
 			(end 14.78125 8.000001)
 			(stroke
@@
 		(fp_arc
 			(start 14.780039 -5.999999)
-			(mid 15.133567 -5.853539)
+			(mid 15.133602 -5.853545)
 			(end 15.280039 -5.499999)
 			(stroke
@@
 		(fp_arc
 			(start 9.03125 8.000001)
-			(mid 8.677729 7.853537)
+			(mid 8.677693 7.853543)
 			(end 8.53125 7.500001)
 			(stroke
@@
 		(fp_arc
 			(start 15.28125 7.500001)
-			(mid 15.134806 7.853571)
+			(mid 15.1348 7.853536)
 			(end 14.78125 8.000001)
 			(stroke
@@
 		(fp_arc
 			(start 14.780039 -5.999999)
-			(mid 15.133567 -5.853539)
+			(mid 15.133602 -5.853545)
 			(end 15.280039 -5.499999)
 			(stroke
@@
 		(fp_arc
 			(start 9.03125 8.000001)
-			(mid 8.677729 7.853537)
+			(mid 8.677693 7.853543)
 			(end 8.53125 7.500001)
 			(stroke
@@
 	(footprint "MountingHole:MountingHole_2.2mm_M2_Pad"
 		(layer "F.Cu")
-		(at 354.202326 78.614934)
+		(at 354.202326 92.901934)
 		(descr "Mounting Hole 2.2mm, M2")
 		(tags "mounting hole 2.2mm m2")
@@
 		(fp_arc
 			(start 53.38125 7.500001)
-			(mid 53.2348 7.853536)
+			(mid 53.234806 7.853571)
 			(end 52.88125 8.000001)
 			(stroke
@@
 		(fp_arc
 			(start 52.880039 -5.999999)
-			(mid 53.233602 -5.853545)
+			(mid 53.233567 -5.853539)
 			(end 53.380039 -5.499999)
 			(stroke
@@
 		(fp_arc
 			(start 47.13125 8.000001)
-			(mid 46.777693 7.853543)
+			(mid 46.777729 7.853537)
 			(end 46.63125 7.500001)
 			(stroke
@@
 		(fp_arc
 			(start 46.63125 -5.499999)
-			(mid 46.777699 -5.853535)
+			(mid 46.777693 -5.853571)
 			(end 47.13125 -5.999999)
 			(stroke
@@
 		(fp_arc
 			(start 6.085176 4.75022)
-			(mid 5.499389 6.164432)
+			(mid 5.499388 6.164432)
 			(end 4.085176 6.75022)
 			(stroke
@@
 		(fp_arc
 			(start 6.085176 4.75022)
-			(mid 5.499389 6.164432)
+			(mid 5.499388 6.164432)
 			(end 4.085176 6.75022)
 			(stroke
@@
 		(fp_arc
 			(start 6.085176 4.75022)
-			(mid 5.499389 6.164432)
+			(mid 5.499388 6.164432)
 			(end 4.085176 6.75022)
 			(stroke
@@
 		(fp_arc
 			(start 6.085176 4.75022)
-			(mid 5.499389 6.164432)
+			(mid 5.499388 6.164432)
 			(end 4.085176 6.75022)
 			(stroke
@@
 		(fp_arc
 			(start 6.085176 4.75022)
-			(mid 5.499389 6.164432)
+			(mid 5.499388 6.164432)
 			(end 4.085176 6.75022)
 			(stroke
@@
 		(fp_arc
 			(start 6.085176 4.75022)
-			(mid 5.499389 6.164432)
+			(mid 5.499388 6.164432)
 			(end 4.085176 6.75022)
 			(stroke
